Commit message: 优化仿真模型, 添加示例配置

File: models/s1/s1.urdf (robot description, URDF)
Before this commit: robot robot_gazebo_s1, 14 links, 13 joints
Joints:
- joint front_wheel_joint: origin xyz=0.616967 0.002805 -0.696785 rpy=0 0 0 -> xyz=0.616967 0 -0.690066 rpy=0 0 0

Commit message: 完成模型地图

File: models/s1/s1.urdf (robot description, URDF)
Before this commit: robot robot_gazebo_s1, 14 links, 13 joints
Joints:
- joint front_wheel_joint: origin xyz=0.616967 0 -0.690066 rpy=0 0 0 -> xyz=0.616967 0 -0.692066 rpy=0 0 0
